Commit message: wheel

File: my_bot/description/robot_core.xacro (robot description, xacro)
@@ -16,4 +16,5 @@
     <link name="base_link">
     </link>
+<!-- chassis link -->
     <joint name="chassis_link" type="fixed">
         <parent link="base_link"/>
@@ -31,3 +32,63 @@
         </visual>
     </link>
+    <!-- left wheel joint-->
+    <joint name = "left_wheel_Joint" type ="continuous">
+        <parent link="base_link"/>
+        <child link="left_wheel"/>
+        <origin xyz="0.0 0.175 0.0" rpy="-${pi/2} 0.0 0.0"/>
+        <axis xyz="0.0 0.0 1"/>
+    </joint>
+    <link name="left_wheel">
+        <!-- <inertial>
+            <origin xyz="0.0 0.0 0.0" rpy="0.0 0.0 0.0"/>
+            <mass value="0.0"/>
+            <inertia ixx="0.0" ixy="0.0" ixz="0.0" iyy="0.0" iyz="0.0" izz="0.0"/>
+        </inertial> -->
+        <visual name="">
+            <origin xyz="0.0 0.0 0.0" rpy="0.0 0.0 0.0"/>
+            <geometry>
+                <geometry>
+                    <cylinder radius="0.05" length="0.04"/>
+                </geometry>
+            </geometry>
+            <material name="white">
+            </material>
+        </visual>
+        <!-- <collision>
+            <origin xyz="0.0 0.0 0.0" rpy="0.0 0.0 0.0"/>
+            <geometry>
+                <box size="0.0 0.0 0.0"/>
+            </geometry>
+        </collision> -->
+    </link>
+    <!-- right wheel joint-->
+    <joint name = "right_wheel_Joint" type ="continuous">
+        <parent link="base_link"/>
+        <child link="right_wheel"/>
+        <origin xyz="0.0 -0.175 0.0" rpy="-${pi/2} 0.0 0.0"/>
+        <axis xyz="0.0 0.0 -1"/>
+    </joint>
+    <link name="right_wheel">
+        <!-- <inertial>
+            <origin xyz="0.0 0.0 0.0" rpy="0.0 0.0 0.0"/>
+            <mass value="0.0"/>
+            <inertia ixx="0.0" ixy="0.0" ixz="0.0" iyy="0.0" iyz="0.0" izz="0.0"/>
+        </inertial> -->
+        <visual name="">
+            <origin xyz="0.0 0.0 0.0" rpy="0.0 0.0 0.0"/>
+            <geometry>
+                <geometry>
+                    <cylinder radius="0.05" length="0.04"/>
+                </geometry>
+            </geometry>
+            <material name="white">
+            </material>
+        </visual>
+        <!-- <collision>
+            <origin xyz="0.0 0.0 0.0" rpy="0.0 0.0 0.0"/>
+            <geometry>
+                <box size="0.0 0.0 0.0"/>
+            </geometry>
+        </collision> -->
+    </link>
 </robot>

Commit message: wheel

File: my_bot/description/robot_core.xacro (robot description, xacro)
@@ -82,6 +82,6 @@
                 </geometry>
             </geometry>
-            <material name="white">
-            </material>
+            <material name="white"/>
+            <!-- </material> -->
         </visual>
         <!-- <collision>

Commit message: wheels

File: my_bot/description/robot_core.xacro (robot description, xacro)
@@ -52,6 +52,6 @@
                 </geometry>
             </geometry>
-            <material name="white">
-            </material>
+            <material name="white"/>
+            <!-- </material> -->
         </visual>
         <!-- <collision>

Commit message: bot urdf robot_core

File: my_bot/description/robot_core.xacro (robot description, xacro)
@@ -1,4 +1,5 @@
 <?xml version="1.0"?>
 <robot xmlns:xacro="http://www.ros.org/wiki/xacro"  >
+    <xacro:include filename="inertial_macros.xacro"/>
     <material name="white">
         <color rgba="1 1 1 1" />
@@ -31,4 +32,13 @@
                 </material>
         </visual>
+        <collision>
+                <origin xyz="0.15 0.0 0.075"/>
+                <geometry>
+                    <box size="0.3 0.3 0.15"/>
+                </geometry>
+        </collision>
+        <xacro:inertial_box mass="0.5" x="0.3" y="0.3" z="0.15">
+            <origin xyz="0.15 0 0.075" rpy="0.0 0.0 0.0"/>
+        </xacro:inertial_box>
     </link>
     <!-- left wheel joint-->
@@ -48,17 +58,17 @@
             <origin xyz="0.0 0.0 0.0" rpy="0.0 0.0 0.0"/>
             <geometry>
-                <geometry>
-                    <cylinder radius="0.05" length="0.04"/>
-                </geometry>
+                <cylinder radius="0.05" length="0.04"/>
             </geometry>
-            <material name="white"/>
-            <!-- </material> -->
+            <material name="blue"/>
         </visual>
-        <!-- <collision>
+        <collision>
             <origin xyz="0.0 0.0 0.0" rpy="0.0 0.0 0.0"/>
             <geometry>
-                <box size="0.0 0.0 0.0"/>
+                <cylinder radius="0.05" length="0.04"/>
             </geometry>
-        </collision> -->
+        </collision>
+        <xacro:inertial_cylinder mass="0.1" length="0.04" radius="0.05">
+            <origin xyz="0.0 0.0 0.0" rpy="0.0 0.0 0.0"/>
+        </xacro:inertial_cylinder>
     </link>
     <!-- right wheel joint-->
@@ -70,25 +80,43 @@
     </joint>
     <link name="right_wheel">
-        <!-- <inertial>
-            <origin xyz="0.0 0.0 0.0" rpy="0.0 0.0 0.0"/>
-            <mass value="0.0"/>
-            <inertia ixx="0.0" ixy="0.0" ixz="0.0" iyy="0.0" iyz="0.0" izz="0.0"/>
-        </inertial> -->
-        <visual name="">
+        <visual>
             <origin xyz="0.0 0.0 0.0" rpy="0.0 0.0 0.0"/>
             <geometry>
-                <geometry>
                     <cylinder radius="0.05" length="0.04"/>
-                </geometry>
             </geometry>
-            <material name="white"/>
-            <!-- </material> -->
+            <material name="blue"/>
         </visual>
-        <!-- <collision>
+        <collision>
             <origin xyz="0.0 0.0 0.0" rpy="0.0 0.0 0.0"/>
             <geometry>
-                <box size="0.0 0.0 0.0"/>
+                    <cylinder radius="0.05" length="0.04"/>
             </geometry>
-        </collision> -->
+        </collision>
+        <xacro:inertial_cylinder mass="0.1" length="0.04" radius="0.05">
+            <origin xyz="0.0 0.0 0.0" rpy="0.0 0.0 0.0"/>
+        </xacro:inertial_cylinder>
+    </link>
+    <!-- CASTER WHEEL LINK -->
+    <joint name="caster_wheel_joint" type="fixed">
+        <parent link="chassis"/>
+        <child link="caster_wheel"/>
+        <origin xyz="0.24 0.0 0.0"/>
+    </joint>
+    <link name="caster_wheel">
+        <visual>
+            <geometry>
+                <sphere radius="0.05"/>
+            </geometry>
+            <material name="back">
+            </material>
+        </visual>
+        <collision>
+            <geometry>
+                <sphere radius="0.05"/>
+            </geometry>
+        </collision>
+        <xacro:inertial_sphere mass="0.1" radius="0.05">
+            <origin xyz="0.0 0.0 0.0" rpy="0.0 0.0 0.0"/>
+        </xacro:inertial_sphere>
     </link>
 </robot>

Commit message: gazebo

File: my_bot/description/robot_core.xacro (robot description, xacro)
@@ -42,4 +42,9 @@
         </xacro:inertial_box>
     </link>
+    <gazebo reference="chassis">
+        <material>
+            Gazebo/White
+        </material>
+    </gazebo>
     <!-- left wheel joint-->
     <joint name = "left_wheel_Joint" type ="continuous">
@@ -72,4 +77,9 @@
         </xacro:inertial_cylinder>
     </link>
+    <gazebo reference="left_wheel">
+        <material>
+            Gazebo/Blue
+        </material>
+    </gazebo>
     <!-- right wheel joint-->
     <joint name = "right_wheel_Joint" type ="continuous">
@@ -97,4 +107,9 @@
         </xacro:inertial_cylinder>
     </link>
+    <gazebo reference="right_wheel">
+        <material>
+            Gazebo/Blue
+        </material>
+    </gazebo>
     <!-- CASTER WHEEL LINK -->
     <joint name="caster_wheel_joint" type="fixed">
@@ -120,3 +135,8 @@
         </xacro:inertial_sphere>
     </link>
+    <gazebo reference="caster_wheel">
+        <material>
+            Gazebo/Black
+        </material>
+    </gazebo>
 </robot>

Commit message: lidar

File: my_bot/description/robot_core.xacro (robot description, xacro)
@@ -13,4 +13,7 @@
     <material name="black">
         <color rgba="0 0 0 1" />
+    </material>
+    <material name="red">
+        <color rgba="1 0 0 1" />
     </material>
 <!-- base link -->

Commit message: slam

File: my_bot/description/robot_core.xacro (robot description, xacro)
@@ -20,4 +20,14 @@
     <link name="base_link">
     </link>
+    <!-- Base footprint link -->
+<joint name="base_footprint_joint" type="fixed">
+    <origin xyz="0.0 0.0 0.0" rpy="0.0 0.0 0.0"/>
+    <parent link="base_link"/>
+    <child link="base_footprint"/>
+    <axis xyz="0.0 0.0 0.0"/>
+    <limit lower="0.0" upper="0.0" effort="0.0" velocity="0.0"/>
+</joint>
+<link name="base_footprint">
+</link>
 <!-- chassis link -->
     <joint name="chassis_link" type="fixed">
