Commit message: latest farthest object problrm is raise and to be unsolved in this commit

File: description/robot_core.xacro (robot description, xacro)
@@ -99,5 +99,5 @@
         <parent link="base_link"/>
         <child link="right_wheel"/>
-        <origin xyz="0.0 -0.175 0.0" rpy="-${pi/2} 0.0 0.0"/>
+        <origin xyz="0.0 -0.175 0.0" rpy="${pi/2} 0.0 0.0"/>
         <axis xyz="0.0 0.0 -1"/>
     </joint>
